File: Hardware/ESP_Wifi_VentilationControll.kicad_pcb (KiCad board)
At the start: 2 copper layers, 52 x 37 mm, 35 parts, among them J1 programming, Q1 2N3904, Q2 2N3904, SW1 RST, SW2 BOOT, U1 LM1117-3.3, U2 ESP-12E, U3 ILD207T_D207, U4 ILD207T_D207, U5 XD-45_MH_MINI

Commit message: added smoothing capacitors
Parts:
- added C2: 100nf, Capacitor_SMD:C_0805_2012Metric, F.Cu at (169.0, 106.5)
- C1: value 330uf -> 1uf; footprint Capacitor_THT:CP_Radial_D8.0mm_P3.50mm -> Capacitor_SMD:C_0805_2012Metric
- moved C1 23.6 mm to (130.0, 109.0), turned to 180 degrees
- moved Q1 3.54 mm to (129.5, 102.0)
- moved Q2 3.54 mm to (129.5, 90.0)
- moved R2 3.54 mm to (129.5, 96.0)
- moved R3 3.54 mm to (129.5, 93.5)
- moved R4 3.54 mm to (129.5, 98.5)
Connections:
- C1 pad 1: VCC -> Net-(C1-Pad1)
- TP11 pad 1: Net-(TP11-Pad1) -> Net-(C1-Pad1)
- U5 pad 1: Net-(TP11-Pad1) -> Net-(C1-Pad1)
Routing:
- net Net-(C1-Pad1): track 0.00 -> 22.3 mm, vias 0 -> 3
- net Net-(TP11-Pad1): track 18.1 -> 0.00 mm, vias 3 -> 0
- net +3V3: track 55.9 -> 65.4 mm
- net GND: track 36.4 -> 44.6 mm
- net Net-(Q1-Pad3): track 64.7 -> 60.6 mm
- net Net-(R2-Pad2): track 9.92 -> 6.61 mm
- net /RTS: track 15.6 -> 18.1 mm
- net /DTR: track 27.7 -> 29.6 mm
- net Net-(Q1-Pad2): track 16.9 -> 17.9 mm

Commit message: added status LED
Parts:
- added D1: RED, LED_SMD:LED_1206_3216Metric, F.Cu at (129.5, 83.5)
- added R14: 1k, Resistor_SMD:R_1206_3216Metric, F.Cu at (129.5, 86.0)
Routing:
- net +3V3: track 65.4 -> 80.5 mm, vias 2 -> 4
- net Net-(D1-Pad1): track 0.00 -> 3.90 mm
- net Net-(Q2-Pad3): track 49.5 -> 53.2 mm
Changed lines of the file:
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@@
   (net 42 "unconnected-(U2-Pad5)")
   (net 43 "Net-(C1-Pad1)")
+  (net 44 "Net-(D1-Pad1)")
   (footprint "ESP8266:ESP-12E_SMD" (layer "F.Cu")
     (at 136.5 89.4125)
@@
     (pad "1" smd roundrect (at 0 0 270) (size 1 2) (layers "F.Cu" "F.Paste" "F.Mask") (roundrect_rratio 0.25)
       (net 23 "Net-(R12-Pad1)") (pinfunction "1") (pintype "passive"))
+  )
+  (footprint "Resistor_SMD:R_1206_3216Metric" (layer "F.Cu")
+    (at 129.5 86)
+    (descr "Resistor SMD 1206 (3216 Metric), square (rectangular) end terminal, IPC_7351 nominal, (Body size source: IPC-SM-782 page 72, https://www.pcb-3d.com/wordpress/wp-content/uploads/ipc-sm-782a_amendment_1_and_2.pdf), generated with kicad-footprint-generator")
+    (tags "resistor")
+    (property "Sheetfile" "ESP_Wifi_VentilationControll.kicad_sch")
+    (property "Sheetname" "")
+    (attr smd)
+    (fp_text reference "R14" (at 3.5 0) (layer "F.SilkS")
+      (effects (font (size 0.5 0.5) (thickness 0.125)))
+    )
+    (fp_text value "1k" (at 0 1.82) (layer "F.Fab")
+      (effects (font (size 1 1) (thickness 0.15)))
+    )
+    (fp_text user "${REFERENCE}" (at 0 0) (layer "F.Fab")
+      (effects (font (size 0.8 0.8) (thickness 0.12)))
+    )
+    (fp_line (start -0.727064 0.91) (end 0.727064 0.91) (layer "F.SilkS") (width 0.12))
+    (fp_line (start -0.727064 -0.91) (end 0.727064 -0.91) (layer "F.SilkS") (width 0.12))
+    (fp_line (start -2.28 1.12) (end -2.28 -1.12) (layer "F.CrtYd") (width 0.05))
+    (fp_line (start 2.28 1.12) (end -2.28 1.12) (layer "F.CrtYd") (width 0.05))
+    (fp_line (start 2.28 -1.12) (end 2.28 1.12) (layer "F.CrtYd") (width 0.05))
+    (fp_line (start -2.28 -1.12) (end 2.28 -1.12) (layer "F.CrtYd") (width 0.05))
+    (fp_line (start 1.6 0.8) (end -1.6 0.8) (layer "F.Fab") (width 0.1))
+    (fp_line (start -1.6 -0.8) (end 1.6 -0.8) (layer "F.Fab") (width 0.1))
+    (fp_line (start -1.6 0.8) (end -1.6 -0.8) (layer "F.Fab") (width 0.1))
+    (fp_line (start 1.6 -0.8) (end 1.6 0.8) (layer "F.Fab") (width 0.1))
+    (pad "1" smd roundrect (at -1.4625 0) (size 1.125 1.75) (layers "F.Cu" "F.Paste" "F.Mask") (roundrect_rratio 0.222222)
+      (net 10 "Net-(Q2-Pad3)") (pintype "passive"))
+    (pad "2" smd roundrect (at 1.4625 0) (size 1.125 1.75) (layers "F.Cu" "F.Paste" "F.Mask") (roundrect_rratio 0.222222)
+      (net 44 "Net-(D1-Pad1)") (pintype "passive"))
+    (model "${KICAD6_3DMODEL_DIR}/Resistor_SMD.3dshapes/R_1206_3216Metric.wrl"
+      (offset (xyz 0 0 0))
+      (scale (xyz 1 1 1))
+      (rotate (xyz 0 0 0))
+    )
+  )
+  (footprint "LED_SMD:LED_1206_3216Metric" (layer "F.Cu")
+    (at 129.5 83.5)
+    (descr "LED SMD 1206 (3216 Metric), square (rectangular) end terminal, IPC_7351 nominal, (Body size source: http://www.tortai-tech.com/upload/download/2011102023233369053.pdf), generated with kicad-footprint-generator")
+    (tags "LED")
+    (property "Sheetfile" "ESP_Wifi_VentilationControll.kicad_sch")
+    (property "Sheetname" "")
+    (attr smd)
+    (fp_text reference "D1" (at 3.5 0) (layer "F.SilkS")
+      (effects (font (size 0.5 0.5) (thickness 0.125)))
+    )
+    (fp_text value "RED" (at 0 1.82) (layer "F.Fab")
+      (effects (font (size 1 1) (thickness 0.15)))
+    )
+    (fp_text user "${REFERENCE}" (at 0 0) (layer "F.Fab")
+      (effects (font (size 0.8 0.8) (thickness 0.12)))
+    )
+    (fp_line (start -2.285 1.135) (end 1.6 1.135) (layer "F.SilkS") (width 0.12))
+    (fp_line (start -2.285 -1.135) (end -2.285 1.135) (layer "F.SilkS") (width 0.12))
+    (fp_line (start 1.6 -1.135) (end -2.285 -1.135) (layer "F.SilkS") (width 0.12))
+    (fp_line (start -2.28 -1.12) (end 2.28 -1.12) (layer "F.CrtYd") (width 0.05))
+    (fp_line (start 2.28 -1.12) (end 2.28 1.12) (layer "F.CrtYd") (width 0.05))
+    (fp_line (start -2.28 1.12) (end -2.28 -1.12) (layer "F.CrtYd") (width 0.05))
+    (fp_line (start 2.28 1.12) (end -2.28 1.12) (layer "F.CrtYd") (width 0.05))
+    (fp_line (start 1.6 -0.8) (end -1.2 -0.8) (layer "F.Fab") (width 0.1))
+    (fp_line (start -1.6 0.8) (end 1.6 0.8) (layer "F.Fab") (width 0.1))
+    (fp_line (start 1.6 0.8) (end 1.6 -0.8) (layer "F.Fab") (width 0.1))
+    (fp_line (start -1.6 -0.4) (end -1.6 0.8) (layer "F.Fab") (width 0.1))
+    (fp_line (start -1.2 -0.8) (end -1.6 -0.4) (layer "F.Fab") (width 0.1))
+    (pad "1" smd roundrect (at -1.4 0) (size 1.25 1.75) (layers "F.Cu" "F.Paste" "F.Mask") (roundrect_rratio 0.2)
+      (net 44 "Net-(D1-Pad1)") (pinfunction "K") (pintype "passive"))
+    (pad "2" smd roundrect (at 1.4 0) (size 1.25 1.75) (layers "F.Cu" "F.Paste" "F.Mask") (roundrect_rratio 0.2)
+      (net 11 "+3V3") (pinfunction "A") (pintype "passive"))
+    (model "${KICAD6_3DMODEL_DIR}/LED_SMD.3dshapes/LED_1206_3216Metric.wrl"
+      (offset (xyz 0 0 0))
+      (scale (xyz 1 1 1))
+      (rotate (xyz 0 0 0))
+    )
   )
   (footprint "Resistor_SMD:R_1206_3216Metric" (layer "F.Cu")
@@
   (via (at 133.8 89.4) (size 0.8) (drill 0.4) (layers "F.Cu" "B.Cu") (net 8))
   (via (at 156.237269 98) (size 0.8) (drill 0.4) (layers "F.Cu" "B.Cu") (net 8))
+  (segment (start 130.5 94.6495) (end 130.5 101.4) (width 0.5) (layer "B.Cu") (net 8))
   (segment (start 156.25 98.012731) (end 156.237269 98) (width 0.5) (layer "B.Cu") (net 8))
-  (segment (start 133.8 89.4) (end 129.5505 93.6495) (width 0.5) (layer "B.Cu") (net 8))
-  (segment (start 129.5 93.6495) (end 129.5 102.4) (width 0.5) (layer "B.Cu") (net 8))
+  (segment (start 130.5 93) (end 130.5 95) (width 0.5) (layer "B.Cu") (net 8))
+  (segment (start 133.8 89.4) (end 133.8 89.7) (width 0.5) (layer "B.Cu") (net 8))
+  (segment (start 130.5 101.4) (end 129.5 102.4) (width 0.5) (layer "B.Cu") (net 8))
+  (segment (start 133.8 89.7) (end 130.5 93) (width 0.5) (layer "B.Cu") (net 8))
   (segment (start 156.25 104.5) (end 156.25 98.012731) (width 0.5) (layer "B.Cu") (net 8))
   (segment (start 130.9625 98.5) (end 129.95048 97.48798) (width 0.5) (layer "F.Cu") (net 9))
@@
   (segment (start 157.5 104.5) (end 157.5 104.75) (width 0.5) (layer "F.Cu") (net 10))
   (segment (start 150.5 97.4125) (end 147.4125 97.4125) (width 0.5) (layer "F.Cu") (net 10))
+  (segment (start 129.5 89.0625) (end 129.5 87.4625) (width 0.5) (layer "F.Cu") (net 10))
   (segment (start 160.6 114.15) (end 160.6 107.85) (width 0.5) (layer "F.Cu") (net 10))
   (segment (start 133.61062 90.412011) (end 132.261109 89.0625) (width 0.5) (layer "F.Cu") (net 10))
@@
   (segment (start 153.5 97.5) (end 153.4125 97.4125) (width 0.5) (layer "F.Cu") (net 10))
   (segment (start 153.4125 97.4125) (end 150.5 97.4125) (width 0.5) (layer "F.Cu") (net 10))
+  (segment (start 129.5 87.4625) (end 128.0375 86) (width 0.5) (layer "F.Cu") (net 10))
   (segment (start 147.4125 97.4125) (end 140.412011 90.412011) (width 0.5) (layer "F.Cu") (net 10))
   (via (at 153.5 97.5) (size 0.8) (drill 0.4) (layers "F.Cu" "B.Cu") (net 10))
@@
   (segment (start 170.849511 101.349511) (end 170 100.5) (width 1) (layer "F.Cu") (net 11))
   (segment (start 129.04952 97.01202) (end 129.04952 98.54952) (width 0.5) (layer "F.Cu") (net 11))
+  (segment (start 130.9 83.5) (end 129.5 83.5) (width 0.5) (layer "F.Cu") (net 11))
   (segment (start 150.5 108.5) (end 155 104) (width 1) (layer "F.Cu") (net 11))
   (segment (start 136.5 103.4125) (end 136.5 106.696377) (width 1) (layer "F.Cu") (net 11))
@@
   (segment (start 170 100.5) (end 169.15 100.5) (width 1) (layer "F.Cu") (net 11))
   (segment (start 139.303623 109.5) (end 143.5 109.5) (width 1) (layer "F.Cu") (net 11))
+  (segment (start 129.10098 96) (end 128.0375 96) (width 0.5) (layer "F.Cu") (net 11))
   (segment (start 158.603964 103.5) (end 162 103.5) (width 1) (layer "F.Cu") (net 11))
   (segment (start 134 103.5) (end 136.4125 103.5) (width 0.5) (layer "F.Cu") (net 11))
   (via (at 150.5 109.5) (size 0.8) (drill 0.4) (layers "F.Cu" "B.Cu") (net 11))
   (via (at 143.5 109.5) (size 0.8) (drill 0.4) (layers "F.Cu" "B.Cu") (net 11))
+  (via (at 129.10098 96) (size 0.8) (drill 0.4) (layers "F.Cu" "B.Cu") (net 11))
+  (via (at 129.5 83.5) (size 0.8) (drill 0.4) (layers "F.Cu" "B.Cu") (net 11))
   (segment (start 150.5 109.5) (end 143.5 109.5) (width 1) (layer "B.Cu") (net 11))
+  (segment (start 129.10098 96) (end 129.5 95.60098) (width 0.5) (layer "B.Cu") (net 11))
+  (segment (start 129.5 95.60098) (end 129.5 83.5) (width 0.5) (layer "B.Cu") (net 11))
   (segment (start 136.5 93.4125) (end 133.55 93.4125) (width 0.5) (layer "F.Cu") (net 12))
   (segment (start 133.55 93.4125) (end 130.9625 96) (width 0.5) (layer "F.Cu") (net 12))
@@
   (segment (start 133 111.5) (end 135 111.5) (width 1) (layer "B.Cu") (net 43))
   (segment (start 142 107.5) (end 142 103) (width 1) (layer "B.Cu") (net 43))
+  (segment (start 130.9625 86) (end 130.6 86) (width 0.5) (layer "F.Cu") (net 44))
+  (segment (start 130.6 86) (end 128.1 83.5) (width 0.5) (layer "F.Cu") (net 44))
   (zone (net 1) (net_name "VCC") (layer "F.Cu") (hatch edge 0.508)
     (connect_pads (clearance 0.508))
